File: ATM90E26_Featherwing.sch (KiCad schematic (older format))
At the start: 59 parts, among them J1 ST-PJ-312, J2 4P-SMD-2.0-90D, J3 4P-SMD-2.0-90D, J4 12V AC, Q1 8.192MHz, U1 ATM90E26, U2 CJT1117-5.0-SOT223

Commit message: Clean out tracks and zones, place parts
Parts:
- C1, C8: footprint AVX-A -> ATM90E26_Featherwing:AVX-A
- C10, C11, C12, C13, C16, C17, C2, C3, C4, C5, C6, C7, C9: footprint C0603 -> ATM90E26_Featherwing:C0603
- C14: footprint 140CLH-1010 -> ATM90E26_Featherwing:140CLH-1010
- C15: footprint 153CLV-0605 -> ATM90E26_Featherwing:153CLV-0605
- CF1, CF2, CS1, I2N_IN1, I2P_IN1, INT1, SCLK1, SI/RX1, SO/TX1, WARN1, ZX1: footprint SMD1,27-2,54 -> ATM90E26_Featherwing:SMD1,27-2,54
- CSMUX1, RXMUX1, TXMUX1: footprint PAD-JUMPER-3-NO_YES_SILK -> ATM90E26_Featherwing:PAD-JUMPER-3-NO_YES_SILK
- D1: footprint SMA-DIODE -> ATM90E26_Featherwing:SMA-DIODE
- D2: footprint SOD-123 -> ATM90E26_Featherwing:SOD-123
- J1: footprint AUDIO6P-SMD-3.5-14.0X6.4X5.0MM -> ATM90E26_Featherwing:AUDIO6P-SMD-3.5-14.0X6.4X5.0MM
- J2, J3: footprint HW4-SMD-2.0-90D -> ATM90E26_Featherwing:HW4-SMD-2.0-90D
- J4: footprint DC_BARREL_JACK_SMD_2MM -> ATM90E26_Featherwing:DC_BARREL_JACK_SMD_2MM
- LOGO1: footprint OSHW-LOGO-M -> ATM90E26_Featherwing:OSHW-LOGO-M
- MMD0, MMD1, USEL1: footprint PAD-JUMPER-3-NO_YES_SILK_FULL_BOX -> ATM90E26_Featherwing:PAD-JUMPER-3-NO_YES_SILK_FULL_BOX
- MS1: footprint FEATHERWING_DIM -> ATM90E26_Featherwing:FEATHERWING_DIM
- PWR1: footprint LED-0603 -> ATM90E26_Featherwing:LED-0603
- Q1: footprint HC49UP -> ATM90E26_Featherwing:HC49UP
- R1, R10, R11, R13, R2, R3, R5, R6, R7, R8, R9: footprint R0603 -> ATM90E26_Featherwing:R0603
- R12: footprint 0805 -> ATM90E26_Featherwing:0805
- SCKMUX1: footprint PAD-JUMPER-2-NO_YES_SILK -> ATM90E26_Featherwing:PAD-JUMPER-2-NO_YES_SILK
- U1: footprint SSOP-28 -> ATM90E26_Featherwing:SSOP-28
- U2: footprint SOT-223 -> ATM90E26_Featherwing:SOT-223

Commit message: Initial autoroute
Parts:
- LOGO1: footprint ATM90E26_Featherwing:OSHW-LOGO-M -> Symbols:OSHW-Logo2_7.3x6mm_Copper
Connections:
- net labels added: 5V_REG, AC_REC, AC_VP
Changed lines of the file:
@@
 F 0 "LOGO1" H 11100 6500 50  0001 C CNN
 F 1 "OSHW-LOGOM" H 11100 6500 50  0001 C CNN
-F 2 "ATM90E26_Featherwing:OSHW-LOGO-M" H 11100 6500 50  0001 C CNN
+F 2 "Symbols:OSHW-Logo2_7.3x6mm_Copper" H 11100 6500 50  0001 C CNN
 F 3 "" H 11100 6500 50  0001 C CNN
 	1    11100 6500
@@
 Wire Notes Line
 	6400 3900 6400 8300
+Text Label 2600 6100 0    50   ~ 0
+AC_VP
+Text Label 3550 6100 0    50   ~ 0
+AC_REC
+Text Label 5000 6100 0    50   ~ 0
+5V_REG
 $EndSCHEMATC

Commit message: Fixed dangling/disconnected nodes
Connections:
- wire segments 190 -> 205
Changed lines of the file:
@@
 	4200 2400 4600 2400
 Connection ~ 6200 1700
-Text Label 6200 1600 0    70   ~ 0
+Text Label 6200 1500 0    70   ~ 0
 CLKOUT
 Wire Wire Line
@@
 Wire Wire Line
 	7150 2600 6970 2600
-Text Label 3415 4860 2    70   ~ 0
-I1N_IN
 Wire Wire Line
 	2550 4700 2550 4520
 Wire Wire Line
 	2550 4520 3250 4520
-Wire Wire Line
-	3250 4520 3250 4860
 Wire Wire Line
 	3250 4860 3580 4860
@@
 PINMUX
 Wire Wire Line
-	2700 1400 3400 1400
-Wire Wire Line
-	3900 1400 4500 1400
-Wire Wire Line
-	2600 3100 3100 3100
-Wire Wire Line
-	2200 1800 2600 1800
-Wire Wire Line
-	2400 3400 3000 3400
-Wire Wire Line
-	3500 1600 3800 1600
+	2700 1400 3300 1400
+Wire Wire Line
+	3900 1400 4000 1400
+Wire Wire Line
+	2600 3100 2850 3100
+Wire Wire Line
+	2200 1800 2450 1800
+Wire Wire Line
+	2400 3400 2600 3400
+Wire Wire Line
+	3500 1600 3650 1600
 Wire Wire Line
 	5800 2100 6200 2100
@@
 	5790 3270 6220 3270
 Wire Wire Line
-	7100 1700 7100 1900
+	7100 1700 7100 1850
 Wire Wire Line
 	7100 1700 7610 1700
@@
 	7610 2930 7610 3030
 Wire Wire Line
-	2400 7000 3700 7000
-Wire Wire Line
-	2400 2300 3100 2300
+	2400 7000 2650 7000
+Wire Wire Line
+	2400 2300 2550 2300
 Wire Wire Line
 	1580 2400 2400 2400
@@
 	1580 2100 1580 2400
 Wire Wire Line
-	3500 1200 3800 1200
-Wire Wire Line
-	3090 5260 3580 5260
+	3500 1200 3650 1200
+Wire Wire Line
+	3090 5260 3250 5260
 Wire Wire Line
 	3700 6100 4050 6100
 Wire Wire Line
-	1580 2100 2900 2100
+	1580 2100 1700 2100
 Wire Notes Line
 	11700 3900 12050 3900
@@
 Text Label 5000 6100 0    50   ~ 0
 5V_REG
+Connection ~ 2450 1800
+Wire Wire Line
+	2450 1800 2600 1800
+Connection ~ 2850 3100
+Wire Wire Line
+	2850 3100 3100 3100
+Connection ~ 2450 2100
+Wire Wire Line
+	2450 2100 2900 2100
+Connection ~ 2200 2100
+Wire Wire Line
+	2200 2100 2450 2100
+Connection ~ 3650 1600
+Wire Wire Line
+	3650 1600 3800 1600
+Connection ~ 4000 1400
+Wire Wire Line
+	4000 1400 4500 1400
+Connection ~ 3300 1400
+Wire Wire Line
+	3300 1400 3400 1400
+Connection ~ 2850 3400
+Wire Wire Line
+	2850 3400 3000 3400
+Connection ~ 2600 3400
+Wire Wire Line
+	2600 3400 2850 3400
+Connection ~ 1700 2100
+Wire Wire Line
+	1700 2100 2200 2100
+Connection ~ 2550 2300
+Wire Wire Line
+	2550 2300 3100 2300
+Connection ~ 2550 2700
+Connection ~ 4950 6100
+Connection ~ 4050 6100
+Connection ~ 2650 7000
+Wire Wire Line
+	2650 7000 3700 7000
+Connection ~ 7100 1850
+Wire Wire Line
+	7100 1850 7100 1900
+Text Label 3415 4860 2    70   ~ 0
+I1N_IN
+Wire Wire Line
+	3250 4520 3250 4860
+Connection ~ 3250 4860
+Connection ~ 3250 5260
+Wire Wire Line
+	3250 5260 3580 5260
+Connection ~ 2200 1800
+Connection ~ 2600 3100
+Connection ~ 3650 1200
+Wire Wire Line
+	3650 1200 3800 1200
+Connection ~ 3900 1400
+Connection ~ 3400 1400
+Connection ~ 3500 1200
+Connection ~ 3800 1200
+Connection ~ 3800 1600
+Connection ~ 3500 1600
 $EndSCHEMATC

Commit message: ERC and connectivity (#1)
* Add no-connect to unused pins

Signed-off-by: Eliot Blennerhassett <eliot@blennerhassett.gen.nz>

* Connect R11 to ground

Signed-off-by: Eliot Blennerhassett <eliot@blennerhassett.gen.nz>

* pcb: connect R11 to ground

Signed-off-by: Eliot Blennerhassett <eliot@blennerhassett.gen.nz>
Connections:
- wire segments 205 -> 206
- no-connect marks 0 -> 21
Changed lines of the file:
@@
 Text Label 9400 3300 2    70   ~ 0
 +3V3
-Wire Wire Line
-	9400 3000 9400 3340
 Text Label 9610 4550 0    24   ~ 0
 +3V3
@@
 Connection ~ 2650 7000
 Wire Wire Line
-	2650 7000 3700 7000
+	2650 7000 2820 7000
 Connection ~ 7100 1850
 Wire Wire Line
@@
 Wire Wire Line
 	3250 5260 3580 5260
-Connection ~ 2200 1800
-Connection ~ 2600 3100
 Connection ~ 3650 1200
 Wire Wire Line
 	3650 1200 3800 1200
-Connection ~ 3900 1400
-Connection ~ 3400 1400
 Connection ~ 3500 1200
 Connection ~ 3800 1200
 Connection ~ 3800 1600
 Connection ~ 3500 1600
+NoConn ~ 10800 3000
+NoConn ~ 10700 3000
+NoConn ~ 10600 3000
+NoConn ~ 10200 3000
+NoConn ~ 10100 3000
+NoConn ~ 9900 3000
+NoConn ~ 9800 3000
+NoConn ~ 9700 3000
+NoConn ~ 9500 3000
+NoConn ~ 9300 3000
+NoConn ~ 2650 5500
+NoConn ~ 2150 5500
+NoConn ~ 1850 4700
+NoConn ~ 2000 6500
+NoConn ~ 10600 1300
+NoConn ~ 10500 1300
+NoConn ~ 10100 1300
+NoConn ~ 9800 1300
+NoConn ~ 9700 1300
+NoConn ~ 2750 4700
+NoConn ~ 10000 3000
+Wire Wire Line
+	9400 3000 9400 3340
+Connection ~ 2820 7000
+Wire Wire Line
+	2820 7000 3700 7000
 $EndSCHEMATC

Commit message: Successfully fabricated and merged with 3-pin stereo (#2)
* Converted to SJ-3525 for current clamp input

* Add stitchig vias

* New gerbers and git ignore of temp files

Signed-off-by: Tisham Dhar <whatnickd@gmail.com>
Parts:
- removed J1: ST-PJ-312, ATM90E26_Featherwing:AUDIO6P-SMD-3.5-14.0X6.4X5.0MM, symbol ATM90E26_Featherwing-eagle-import:AUDIO-JACK-6P-SMD(ST-PJ-312)
- added J1: AudioJack3, Connector_Audio:Jack_3.5mm_CUI_SJ-3523-SMT_Horizontal, symbol Connector:AudioJack3
Connections:
- wire segments 206 -> 203
- no-connect marks 21 -> 17
Changed lines of the file:
@@
 Text Label 3580 5260 2    70   ~ 0
 I1P_IN
-Wire Wire Line
-	1950 5500 1950 5650
-Wire Wire Line
-	1950 5650 3090 5650
-Wire Wire Line
-	3090 5650 3090 5260
 Text Label 6970 2600 0    70   ~ 0
 I1N_IN
 Wire Wire Line
 	7150 2600 6970 2600
-Wire Wire Line
-	2550 4700 2550 4520
-Wire Wire Line
-	2550 4520 3250 4520
-Wire Wire Line
-	3250 4860 3580 4860
 Connection ~ 7100 1300
 Text Label 6700 1300 0    70   ~ 0
@@
 	1    5660 6700
 	0    1    1    0
-$EndComp
-$Comp
-L ATM90E26_Featherwing-eagle-import:AUDIO-JACK-6P-SMD(ST-PJ-312) J1
-U 1 0 80165544
-P 2300 5100
-F 0 "J1" H 2050 5350 42  0000 L BNN
-F 1 "ST-PJ-312" H 2200 4800 42  0000 L BNN
-F 2 "ATM90E26_Featherwing:AUDIO6P-SMD-3.5-14.0X6.4X5.0MM" H 2300 5100 50  0001 C CNN
-F 3 "" H 2300 5100 50  0001 C CNN
-	1    2300 5100
-	-1   0    0    1
 $EndComp
 $Comp
@@
 Wire Wire Line
 	3500 1200 3650 1200
-Wire Wire Line
-	3090 5260 3250 5260
 Wire Wire Line
 	3700 6100 4050 6100
@@
 Text Label 3415 4860 2    70   ~ 0
 I1N_IN
-Wire Wire Line
-	3250 4520 3250 4860
-Connection ~ 3250 4860
 Connection ~ 3250 5260
 Wire Wire Line
@@
 NoConn ~ 9500 3000
 NoConn ~ 9300 3000
-NoConn ~ 2650 5500
-NoConn ~ 2150 5500
-NoConn ~ 1850 4700
 NoConn ~ 2000 6500
 NoConn ~ 10600 1300
@@
 NoConn ~ 9800 1300
 NoConn ~ 9700 1300
-NoConn ~ 2750 4700
 NoConn ~ 10000 3000
 Wire Wire Line
@@
 Wire Wire Line
 	2820 7000 3700 7000
+$Comp
+L Connector:AudioJack3 J1
+U 1 1 5D0721CB
+P 2700 5055
+F 0 "J1" H 2680 5380 50  0000 C CNN
+F 1 "AudioJack3" H 2680 5289 50  0000 C CNN
+F 2 "Connector_Audio:Jack_3.5mm_CUI_SJ-3523-SMT_Horizontal" H 2700 5055 50  0001 C CNN
+F 3 "~" H 2700 5055 50  0001 C CNN
+	1    2700 5055
+	1    0    0    -1
+$EndComp
+Wire Wire Line
+	2900 4860 2900 4955
+Wire Wire Line
+	2900 4860 3250 4860
+Connection ~ 3250 4860
+Wire Wire Line
+	3250 4860 3580 4860
+Wire Wire Line
+	2900 5155 2900 5260
+Wire Wire Line
+	2900 5260 3250 5260
 $EndSCHEMATC

Commit message: Upgrade to KiCAD 5 and add iBOM
Signed-off-by: Tisham Dhar <whatnickd@gmail.com>
Parts:
- C1, C8: manf# (none) -> TAJA106K010RNJV
- C10, C13, C4, C5: manf# (none) -> GCJ188R71H333KA12D
- C15: manf# (none) -> EMVE160ADA101MF55G
- C16, C17, C2, C6, C9: manf# (none) -> GCJ188R71H104KA12D
- C3, C7: manf# (none) -> GCJ188R91E334MA01J
- CF1, CF2, CS1, CSMUX1, I2N_IN1, I2P_IN1, INT1, LOGO1, MMD0, MMD1, MS1, RXMUX1, SCKMUX1, SCLK1, SI/RX1, SO/TX1, TXMUX1, USEL1, WARN1, ZX1: DNP (none) -> (none)
- J1: manf# (none) -> SJ-3523-SMT-TR
- R13, R2, R3, R6, R9: manf# (none) -> CRT0603-FY-1001ELF

Commit message: Add full iBOM
Signed-off-by: Tisham Dhar <whatnickd@gmail.com>
Parts:
- C11, C12: manf# (none) -> C0603C270F4HACTU
- C14: manf# (none) -> UWT1H221MNL1GS
- D1: manf# (none) -> VS-MBRA140-M3/5AT
- D2: manf# (none) -> MBR120VLSFT3G
- J2, J3, R11: DNP (none) -> (none)
- J4: manf# (none) -> PJ-002AH-SMT-TR
- PWR1: manf# (none) -> LTST-C194TGKT
- Q1: manf# (none) -> ABLS-8.192MHZ-B2-T
- R1, R5: manf# (none) -> CRT0603-FY-1000ELF
- R10: manf# (none) -> CRT0603-FY-1003ELF
- R12: manf# (none) -> RT0805FRE0712RL
- R7, R8: manf# (none) -> CRCW06032R40FKEA
- U1: manf# (none) -> ATM90E26-YU-B
- U2: manf# (none) -> NCP1117ST33T3G
Changed lines of the file:
@@
 F 2 "ATM90E26_Featherwing:SSOP-28" H 3600 2600 50  0001 C CNN
 F 3 "" H 3600 2600 50  0001 C CNN
+F 4 "ATM90E26-YU-B" H 3600 2600 50  0001 C CNN "manf#"
 	1    3600 2600
 	1    0    0    -1
@@
 F 2 "ATM90E26_Featherwing:HC49UP" H 6000 1700 50  0001 C CNN
 F 3 "" H 6000 1700 50  0001 C CNN
+F 4 "ABLS-8.192MHZ-B2-T" H 6000 1700 50  0001 C CNN "manf#"
 	1    6000 1700
 	1    0    0    -1
@@
 F 2 "ATM90E26_Featherwing:C0603" H 5800 1900 50  0001 C CNN
 F 3 "" H 5800 1900 50  0001 C CNN
+F 4 "C0603C270F4HACTU" H 5800 1900 50  0001 C CNN "manf#"
 	1    5800 1900
 	0    1    1    0
@@
 F 2 "ATM90E26_Featherwing:C0603" H 6200 1900 50  0001 C CNN
 F 3 "" H 6200 1900 50  0001 C CNN
+F 4 "C0603C270F4HACTU" H 6200 1900 50  0001 C CNN "manf#"
 	1    6200 1900
 	0    1    1    0
@@
 F 2 "ATM90E26_Featherwing:R0603" H 7100 1500 50  0001 C CNN
 F 3 "" H 7100 1500 50  0001 C CNN
+F 4 "CRCW06032R40FKEA" H 7100 1500 50  0001 C CNN "manf#"
 	1    7100 1500
 	0    1    1    0
@@
 F 2 "ATM90E26_Featherwing:R0603" H 7100 2000 50  0001 C CNN
 F 3 "" H 7100 2000 50  0001 C CNN
+F 4 "CRCW06032R40FKEA" H 7100 2000 50  0001 C CNN "manf#"
 	1    7100 2000
 	0    1    1    0
@@
 F 2 "ATM90E26_Featherwing:R0603" H 7300 2600 50  0001 C CNN
 F 3 "" H 7300 2600 50  0001 C CNN
+F 4 "CRT0603-FY-1000ELF" H 7300 2600 50  0001 C CNN "manf#"
 	1    7300 2600
 	-1   0    0    1
@@
 F 2 "ATM90E26_Featherwing:R0603" H 7300 3400 50  0001 C CNN
 F 3 "" H 7300 3400 50  0001 C CNN
+F 4 "CRT0603-FY-1000ELF" H 7300 3400 50  0001 C CNN "manf#"
 	1    7300 3400
 	-1   0    0    1
@@
 F 2 "ATM90E26_Featherwing:DC_BARREL_JACK_SMD_2MM" H 1800 6500 50  0001 C CNN
 F 3 "" H 1800 6500 50  0001 C CNN
+F 4 "PJ-002AH-SMT-TR" H 1800 6500 50  0001 C CNN "manf#"
 	1    1800 6500
 	1    0    0    -1
@@
 F 2 "ATM90E26_Featherwing:R0603" H 2820 6450 50  0001 C CNN
 F 3 "" H 2820 6450 50  0001 C CNN
+F 4 "CRT0603-FY-1003ELF" H 2820 6450 50  0001 C CNN "manf#"
 	1    2820 6450
 	0    1    1    0
@@
 F 2 "ATM90E26_Featherwing:R0603" H 2820 6850 50  0001 C CNN
 F 3 "" H 2820 6850 50  0001 C CNN
+F 4 " " H 2820 6850 50  0001 C CNN "DNP"
 	1    2820 6850
 	0    1    1    0
@@
 F 2 "ATM90E26_Featherwing:SMA-DIODE" H 3100 6100 50  0001 C CNN
 F 3 "" H 3100 6100 50  0001 C CNN
+F 4 "" H 3100 6100 50  0001 C CNN "DNP"
+F 5 "VS-MBRA140-M3/5AT" H 3100 6100 50  0001 C CNN "manf#"
 	1    3100 6100
 	1    0    0    -1
@@
 F 2 "ATM90E26_Featherwing:SOT-223" H 4500 6100 50  0001 C CNN
 F 3 "" H 4500 6100 50  0001 C CNN
+F 4 "NCP1117ST33T3G" H 4500 6100 50  0001 C CNN "manf#"
 	1    4500 6100
 	1    0    0    -1
@@
 F 2 "ATM90E26_Featherwing:140CLH-1010" H 3700 6400 50  0001 C CNN
 F 3 "" H 3700 6400 50  0001 C CNN
+F 4 "UWT1H221MNL1GS" H 3700 6400 50  0001 C CNN "manf#"
 	1    3700 6400
 	1    0    0    -1
@@
 F 2 "ATM90E26_Featherwing:HW4-SMD-2.0-90D" H 9200 4600 50  0001 C CNN
 F 3 "" H 9200 4600 50  0001 C CNN
+F 4 " " H 9200 4600 50  0001 C CNN "DNP"
 	1    9200 4600
 	-1   0    0    1
@@
 F 2 "ATM90E26_Featherwing:SOD-123" H 5460 6100 50  0001 C CNN
 F 3 "" H 5460 6100 50  0001 C CNN
+F 4 "" H 5460 6100 50  0001 C CNN "DNP"
+F 5 "MBR120VLSFT3G" H 5460 6100 50  0001 C CNN "manf#"
 	1    5460 6100
 	1    0    0    -1
@@
 F 2 "ATM90E26_Featherwing:LED-0603" H 5660 6700 50  0001 C CNN
 F 3 "" H 5660 6700 50  0001 C CNN
+F 4 "" H 5660 6700 50  0001 C CNN "DNP"
+F 5 "LTST-C194TGKT" H 5660 6700 50  0001 C CNN "manf#"
 	1    5660 6700
 	0    1    1    0
@@
 F 2 "ATM90E26_Featherwing:0805" H 3250 5060 50  0001 C CNN
 F 3 "" H 3250 5060 50  0001 C CNN
+F 4 "RT0805FRE0712RL" H 3250 5060 50  0001 C CNN "manf#"
 	1    3250 5060
 	0    -1   -1   0
@@
 F 2 "ATM90E26_Featherwing:HW4-SMD-2.0-90D" H 7700 4600 50  0001 C CNN
 F 3 "" H 7700 4600 50  0001 C CNN
+F 4 " " H 7700 4600 50  0001 C CNN "DNP"
 	1    7700 4600
 	-1   0    0    1
